Commit message: migrate to gazebo sim

File: description/diffbot/urdf/diffbot_description.urdf.xacro (robot description, xacro)
@@ -51,5 +51,5 @@
       <axis xyz="0 1 0"/>
       <dynamics damping="0.05"/>
-      <limit effort="100" velocity="1.0"/>
+      <limit effort="100" velocity="20.0"/>
     </joint>
     <!-- left wheel Link -->
@@ -83,5 +83,5 @@
       <axis xyz="0 1 0"/>
       <dynamics damping="0.05"/>
-      <limit effort="100" velocity="1.0"/>
+      <limit effort="100" velocity="20.0"/>
     </joint>
     <!-- right wheel Link -->

File: description/ros2_control/diffbot.ros2_control.xacro (robot description, xacro)
@@ -1,5 +1,5 @@
 <?xml version="1.0"?>
 <robot xmlns:xacro="http://www.ros.org/wiki/xacro">
-  <xacro:macro name="diffbot_ros2_control" params="name prefix use_hardware use_gazebo_classic">
+  <xacro:macro name="diffbot_ros2_control" params="name prefix use_hardware use_gazebo_classic use_gz_sim">
     <ros2_control name="${name}" type="system">
       <xacro:if value="${use_gazebo_classic}">
@@ -8,5 +8,10 @@
         </hardware>
       </xacro:if>
-      <xacro:unless value="${use_gazebo_classic}">
+      <xacro:if value="${use_gz_sim}">
+        <hardware>
+          <plugin>gz_ros2_control/GazeboSimSystem</plugin>
+        </hardware>
+      </xacro:if>
+      <xacro:unless value="${use_gazebo_classic or use_gz_sim}">
       <xacro:if value="${use_hardware}">
         <hardware>
@@ -49,4 +54,15 @@
         <state_interface name="velocity"/>
       </joint>
+      <xacro:if value="${use_gz_sim}">
+        <!-- Gazebo Sim: publish passive caster joints so robot_state_publisher can build full TF tree. -->
+        <joint name="${prefix}caster_frontal_wheel_joint">
+          <state_interface name="position"/>
+          <state_interface name="velocity"/>
+        </joint>
+        <joint name="${prefix}caster_rear_wheel_joint">
+          <state_interface name="position"/>
+          <state_interface name="velocity"/>
+        </joint>
+      </xacro:if>
     </ros2_control>
   </xacro:macro>

File: description/urdf/diffbot.urdf.xacro (robot description, xacro)
@@ -5,4 +5,5 @@
   <xacro:arg name="use_hardware" default="false" />
   <xacro:arg name="use_gazebo_classic" default="false" />
+  <xacro:arg name="use_gz_sim" default="false" />
   <xacro:include filename="$(find vmxpi_ros2)/description/diffbot/urdf/diffbot_description.urdf.xacro" />
   <!-- Import Rviz colors -->
@@ -15,5 +16,6 @@
     prefix="$(arg prefix)"
     use_hardware="$(arg use_hardware)"
-    use_gazebo_classic="$(arg use_gazebo_classic)"/>
+    use_gazebo_classic="$(arg use_gazebo_classic)"
+    use_gz_sim="$(arg use_gz_sim)"/>
   <xacro:if value="$(arg use_gazebo_classic)">
     <!-- Import Gazebo Classic definitions + plugin -->
@@ -21,3 +23,8 @@
     <xacro:diffbot_gazebo prefix="$(arg prefix)"/>
   </xacro:if>
+  <xacro:if value="$(arg use_gz_sim)">
+    <!-- Import Gazebo Sim definitions + plugin -->
+    <xacro:include filename="$(find vmxpi_ros2)/description/gz/diffbot.gz.xacro" />
+    <xacro:diffbot_gz prefix="$(arg prefix)"/>
+  </xacro:if>
 </robot>

Commit message: rename the project

File: description/diffbot/urdf/diffbot_description.urdf.xacro (robot description, xacro)
@@ -171,5 +171,5 @@
           <origin rpy="0 0 0" xyz="0 0 0"/>
           <geometry>
-            <mesh filename="package://vmxpi_ros2/description/meshes/sensors/hokuyo_urg_04lx.dae" scale="1.0 1.0 1.0"/>
+            <mesh filename="package://studica_vmxpi_ros2/description/meshes/sensors/hokuyo_urg_04lx.dae" scale="1.0 1.0 1.0"/>
             <!-- <cylinder length="0.1" radius="0.05"/> -->
           </geometry>
@@ -178,5 +178,5 @@
           <origin rpy="0 0 0" xyz="0 0 0"/>
           <geometry>
-            <mesh filename="package://vmxpi_ros2/description/meshes/sensors/hokuyo_urg_04lx.dae" scale="1.0 1.0 1.0"/>
+            <mesh filename="package://studica_vmxpi_ros2/description/meshes/sensors/hokuyo_urg_04lx.dae" scale="1.0 1.0 1.0"/>
             <!-- <cylinder length="0.1" radius="0.05"/> -->
           </geometry>

File: description/gazebo/diffbot.gazebo.xacro (robot description, xacro)
@@ -9,5 +9,5 @@
     <gazebo>
       <plugin filename="libgazebo_ros2_control.so" name="gazebo_ros2_control">
-        <parameters>$(find vmxpi_ros2)/config/diffbot_controllers.yaml</parameters>
+        <parameters>$(find studica_vmxpi_ros2)/config/diffbot_controllers.yaml</parameters>
       </plugin>
     </gazebo>

File: description/gz/diffbot.gz.xacro (robot description, xacro)
@@ -5,5 +5,5 @@
     <gazebo>
       <plugin filename="gz_ros2_control-system" name="gz_ros2_control::GazeboSimROS2ControlPlugin">
-        <parameters>$(find vmxpi_ros2)/config/diffbot_controllers.yaml</parameters>
+        <parameters>$(find studica_vmxpi_ros2)/config/diffbot_controllers.yaml</parameters>
       </plugin>
     </gazebo>

File: description/ros2_control/diffbot.ros2_control.xacro (robot description, xacro)
@@ -16,5 +16,5 @@
       <xacro:if value="${use_hardware}">
         <hardware>
-          <plugin>vmxpi_ros2/TitanSystemHardware</plugin>
+          <plugin>studica_vmxpi_ros2/TitanSystemHardware</plugin>
           <param name="can_id">42</param>
           <param name="motor_freq">15600</param>
@@ -38,5 +38,5 @@
         <xacro:unless value="${use_hardware}">
           <hardware>
-            <plugin>vmxpi_ros2/DiffBotSystemHardware</plugin>
+            <plugin>studica_vmxpi_ros2/DiffBotSystemHardware</plugin>
             <param name="example_param_hw_start_duration_sec">0</param>
             <param name="example_param_hw_stop_duration_sec">3.0</param>

File: description/urdf/diffbot.urdf.xacro (robot description, xacro)
@@ -6,9 +6,9 @@
   <xacro:arg name="use_gazebo_classic" default="false" />
   <xacro:arg name="use_gz_sim" default="false" />
-  <xacro:include filename="$(find vmxpi_ros2)/description/diffbot/urdf/diffbot_description.urdf.xacro" />
+  <xacro:include filename="$(find studica_vmxpi_ros2)/description/diffbot/urdf/diffbot_description.urdf.xacro" />
   <!-- Import Rviz colors -->
-  <xacro:include filename="$(find vmxpi_ros2)/description/diffbot/urdf/diffbot.materials.xacro" />
+  <xacro:include filename="$(find studica_vmxpi_ros2)/description/diffbot/urdf/diffbot.materials.xacro" />
   <!-- Import diffbot ros2_control description -->
-  <xacro:include filename="$(find vmxpi_ros2)/description/ros2_control/diffbot.ros2_control.xacro" />
+  <xacro:include filename="$(find studica_vmxpi_ros2)/description/ros2_control/diffbot.ros2_control.xacro" />
   <xacro:diffbot prefix="$(arg prefix)" />
   <xacro:diffbot_ros2_control
@@ -20,10 +20,10 @@
   <xacro:if value="$(arg use_gazebo_classic)">
     <!-- Import Gazebo Classic definitions + plugin -->
-    <xacro:include filename="$(find vmxpi_ros2)/description/gazebo/diffbot.gazebo.xacro" />
+    <xacro:include filename="$(find studica_vmxpi_ros2)/description/gazebo/diffbot.gazebo.xacro" />
     <xacro:diffbot_gazebo prefix="$(arg prefix)"/>
   </xacro:if>
   <xacro:if value="$(arg use_gz_sim)">
     <!-- Import Gazebo Sim definitions + plugin -->
-    <xacro:include filename="$(find vmxpi_ros2)/description/gz/diffbot.gz.xacro" />
+    <xacro:include filename="$(find studica_vmxpi_ros2)/description/gz/diffbot.gz.xacro" />
     <xacro:diffbot_gz prefix="$(arg prefix)"/>
   </xacro:if>

Commit message: imu sensor working

File: description/diffbot/urdf/diffbot_description.urdf.xacro (robot description, xacro)
@@ -202,4 +202,12 @@
         <child link="${prefix}laser_scan_frame"/>
       </joint>
+      <link name="${prefix}imu_link">
+        <origin rpy="0 0 0" xyz="0 0 0"/>
+      </link>
+      <joint name="${prefix}imu_link_joint" type="fixed">
+        <origin rpy="0 0 0" xyz="0 0 0"/>
+        <parent link="${prefix}chassis_link"/>
+        <child link="${prefix}imu_link"/>
+      </joint>
   </xacro:macro>
 </robot>

File: description/ros2_control/diffbot.ros2_control.xacro (robot description, xacro)
@@ -22,4 +22,5 @@
           <param name="wheel_radius">0.05</param>
           <param name="speed_scale">0.5</param>
+          <param name="max_wheel_angular_velocity_rad_s">20.0</param>
           <param name="left_front_motor">2</param>
           <param name="left_rear_motor">3</param>
@@ -54,4 +55,18 @@
         <state_interface name="velocity"/>
       </joint>
+      <xacro:if value="${use_hardware and not use_gazebo_classic and not use_gz_sim}">
+        <sensor name="imu_sensor">
+          <state_interface name="orientation.x"/>
+          <state_interface name="orientation.y"/>
+          <state_interface name="orientation.z"/>
+          <state_interface name="orientation.w"/>
+          <state_interface name="angular_velocity.x"/>
+          <state_interface name="angular_velocity.y"/>
+          <state_interface name="angular_velocity.z"/>
+          <state_interface name="linear_acceleration.x"/>
+          <state_interface name="linear_acceleration.y"/>
+          <state_interface name="linear_acceleration.z"/>
+        </sensor>
+      </xacro:if>
       <xacro:if value="${use_gz_sim}">
         <!-- Gazebo Sim: publish passive caster joints so robot_state_publisher can build full TF tree. -->
