Commit message: fix imu in sim

File: description/gazebo/diffbot.gazebo.xacro (robot description, xacro)
@@ -77,4 +77,8 @@
       <material>Gazebo/White</material>
     </gazebo>
+    <!-- Lidar mesh color override (mesh can appear white in Gazebo if Collada materials are not resolved). -->
+    <gazebo reference="${prefix}laser_model_link">
+      <material>Gazebo/Grey</material>
+    </gazebo>
     <gazebo reference="${prefix}laser_scan_frame">
       <sensor name="sensor_ray" type="ray">

File: description/gz/diffbot.gz.xacro (robot description, xacro)
@@ -1,11 +1,32 @@
 <?xml version="1.0"?>
 <robot xmlns:xacro="http://ros.org/wiki/xacro">
-  <xacro:macro name="diffbot_gz" params="prefix">
+  <xacro:macro name="diffbot_gz" params="prefix gz_version">
     <!-- ros2_control plugin for Gazebo Sim -->
-    <gazebo>
-      <plugin filename="gz_ros2_control-system" name="gz_ros2_control::GazeboSimROS2ControlPlugin">
-        <parameters>$(find studica_vmxpi_ros2)/config/diffbot_controllers.yaml</parameters>
-      </plugin>
-    </gazebo>
+    <xacro:if value="${int(gz_version) &lt; 7}">
+      <gazebo>
+        <plugin filename="ign_ros2_control-system" name="gz_ros2_control::GazeboSimROS2ControlPlugin">
+          <controller_manager_name>controller_manager</controller_manager_name>
+          <robot_param>robot_description</robot_param>
+          <robot_param_node>robot_state_publisher</robot_param_node>
+          <ros>
+            <namespace>/</namespace>
+          </ros>
+          <parameters>$(find studica_vmxpi_ros2)/config/diffbot_controllers.yaml</parameters>
+        </plugin>
+      </gazebo>
+    </xacro:if>
+    <xacro:if value="${int(gz_version) &gt;= 7}">
+      <gazebo>
+        <plugin filename="gz_ros2_control-system" name="gz_ros2_control::GazeboSimROS2ControlPlugin">
+          <controller_manager_name>controller_manager</controller_manager_name>
+          <robot_param>robot_description</robot_param>
+          <robot_param_node>robot_state_publisher</robot_param_node>
+          <ros>
+            <namespace>/</namespace>
+          </ros>
+          <parameters>$(find studica_vmxpi_ros2)/config/diffbot_controllers.yaml</parameters>
+        </plugin>
+      </gazebo>
+    </xacro:if>
     <!-- Base Link -->
     <gazebo reference="${prefix}chassis_link">
@@ -43,4 +64,8 @@
       <mu2>0.001</mu2>
       <material>Gazebo/White</material>
+    </gazebo>
+    <!-- Lidar mesh color override (mesh can appear white in Gazebo if Collada materials are not resolved). -->
+    <gazebo reference="${prefix}laser_model_link">
+      <material>Gazebo/Grey</material>
     </gazebo>
     <!-- Lidar publishes on Gazebo topic /scan; ros_gz_bridge forwards to ROS /scan -->

File: description/ros2_control/diffbot.ros2_control.xacro (robot description, xacro)
@@ -79,4 +79,17 @@
           <state_interface name="velocity"/>
         </joint>
+        <!-- Expose IMU state interfaces in sim so imu_sensor_broadcaster can publish /imu. -->
+        <sensor name="imu_sensor">
+          <state_interface name="orientation.x"/>
+          <state_interface name="orientation.y"/>
+          <state_interface name="orientation.z"/>
+          <state_interface name="orientation.w"/>
+          <state_interface name="angular_velocity.x"/>
+          <state_interface name="angular_velocity.y"/>
+          <state_interface name="angular_velocity.z"/>
+          <state_interface name="linear_acceleration.x"/>
+          <state_interface name="linear_acceleration.y"/>
+          <state_interface name="linear_acceleration.z"/>
+        </sensor>
       </xacro:if>
     </ros2_control>

File: description/urdf/diffbot.urdf.xacro (robot description, xacro)
@@ -6,4 +6,5 @@
   <xacro:arg name="use_gazebo_classic" default="false" />
   <xacro:arg name="use_gz_sim" default="false" />
+  <xacro:arg name="gz_version" default="8" />
   <xacro:include filename="$(find studica_vmxpi_ros2)/description/diffbot/urdf/diffbot_description.urdf.xacro" />
   <!-- Import Rviz colors -->
@@ -26,5 +27,5 @@
     <!-- Import Gazebo Sim definitions + plugin -->
     <xacro:include filename="$(find studica_vmxpi_ros2)/description/gz/diffbot.gz.xacro" />
-    <xacro:diffbot_gz prefix="$(arg prefix)"/>
+    <xacro:diffbot_gz prefix="$(arg prefix)" gz_version="$(arg gz_version)"/>
   </xacro:if>
 </robot>
