Commit message: refactor: simplify bringup and profile workflow for maintainability

File: description/gazebo/robot.gazebo.xacro (robot description, xacro)
@@ -20,6 +20,6 @@
         <plugin name="gazebo_joint_state_broadcaster" filename="libgazebo_ros_joint_state_publisher.so">
           <update_rate>50</update_rate>
-          <joint_name>${prefix}caster_frontal_wheel_joint</joint_name>
-          <joint_name>${prefix}caster_rear_wheel_joint</joint_name>
+          <joint_name>${prefix}caster_left_wheel_joint</joint_name>
+          <joint_name>${prefix}caster_right_wheel_joint</joint_name>
         </plugin>
       </gazebo>
@@ -52,5 +52,5 @@
         <material>Gazebo/Black</material>
       </gazebo>
-      <gazebo reference="${prefix}caster_frontal_wheel">
+      <gazebo reference="${prefix}caster_left_wheel">
         <kp>1e6</kp>
         <kd>1e4</kd>
@@ -63,5 +63,5 @@
         <material>Gazebo/Green</material>
       </gazebo>
-      <gazebo reference="${prefix}caster_rear_wheel">
+      <gazebo reference="${prefix}caster_right_wheel">
         <kp>1e6</kp>
         <kd>1e4</kd>

File: description/gz/robot.gz.xacro (robot description, xacro)
@@ -63,17 +63,17 @@
         <!-- <material>Gazebo/Black</material> -->
       </gazebo>
-      <gazebo reference="${prefix}caster_frontal_wheel">
+      <gazebo reference="${prefix}caster_left_wheel">
         <kp>1e6</kp>
         <kd>1e4</kd>
         <mu1>0.001</mu1>
         <mu2>0.001</mu2>
-        <material>Gazebo/Green</material>
+        <!-- <material>Gazebo/Green</material> -->
       </gazebo>
-      <gazebo reference="${prefix}caster_rear_wheel">
+      <gazebo reference="${prefix}caster_right_wheel">
         <kp>1e6</kp>
         <kd>1e4</kd>
         <mu1>0.001</mu1>
         <mu2>0.001</mu2>
-        <material>Gazebo/White</material>
+        <!-- <material>Gazebo/White</material> -->
       </gazebo>
     </xacro:if>
@@ -130,6 +130,6 @@
           </scan>
           <range>
-            <min>0.1</min>
-            <max>5.0</max>
+            <min>0.5</min>
+            <max>8.0</max>
             <resolution>0.01</resolution>
           </range>

File: description/robot/urdf/robot_description.urdf.xacro (robot description, xacro)
@@ -14,6 +14,6 @@
     <xacro:if value="${wheel_layout_resolved == 'diff'}">
       <xacro:property name="robot_frame_mesh_file" value="package://studica_vmxpi_ros2/description/meshes/frames/robot_frame_4wd.dae"/>
-      <xacro:property name="left_wheel_mesh_file" value="package://studica_vmxpi_ros2/description/meshes/wheels/76249RW.dae"/>
-      <xacro:property name="right_wheel_mesh_file" value="package://studica_vmxpi_ros2/description/meshes/wheels/76249RW.dae"/>
+      <xacro:property name="left_wheel_mesh_file" value="package://studica_vmxpi_ros2/description/meshes/wheels/drive_wheel.dae"/>
+      <xacro:property name="right_wheel_mesh_file" value="package://studica_vmxpi_ros2/description/meshes/wheels/drive_wheel.dae"/>
     </xacro:if>
     <xacro:if value="${wheel_layout_resolved == 'diff_4wd'}">
@@ -68,5 +68,5 @@
         <parent link="${prefix}chassis_link"/>
         <child link="${prefix}left_wheel"/>
-        <origin xyz="0 ${base_width/2} ${wheel_z_offset}" rpy="0 0 0"/>
+        <origin xyz="${base_length/2} ${base_width/2} ${wheel_z_offset}" rpy="0 0 0"/>
         <axis xyz="0 1 0"/>
         <dynamics damping="0.05"/>
@@ -100,5 +100,5 @@
         <parent link="${prefix}chassis_link"/>
         <child link="${prefix}right_wheel"/>
-        <origin xyz="0 -${base_width/2} ${wheel_z_offset}" rpy="0 0 0"/>
+        <origin xyz="${base_length/2} -${base_width/2} ${wheel_z_offset}" rpy="0 0 0"/>
         <axis xyz="0 1 0"/>
         <dynamics damping="0.05"/>
@@ -129,58 +129,66 @@
         </inertial>
       </link>
-      <joint name="${prefix}caster_frontal_wheel_joint" type="continuous">
-        <parent link="${prefix}chassis_link"/>
-        <child link="${prefix}caster_frontal_wheel"/>
-        <origin xyz="${base_width/2 - caster_wheel_radius} 0 ${wheel_z_offset}" rpy="0 0 0"/>
-      </joint>
-      <link name="${prefix}caster_frontal_wheel">
-        <collision>
-          <origin xyz="0 0 0" rpy="0 0 0"/>
-          <geometry>
-            <sphere radius="${caster_wheel_radius}"/>
-          </geometry>
-        </collision>
-        <visual>
-          <origin xyz="0 0 0" rpy="0 0 0"/>
-          <geometry>
-            <sphere radius="${caster_wheel_radius}"/>
-          </geometry>
-          <material name="green"/>
-        </visual>
-        <inertial>
-          <origin xyz="0 0 0" rpy="0 0 0"/>
-          <mass value="${caster_wheel_mass}"/>
-          <inertia
-            ixx="${caster_wheel_mass * 0.4 * (caster_wheel_radius * caster_wheel_radius)}" ixy="0.0" ixz="0.0"
-            iyy="${caster_wheel_mass * 0.4 * (caster_wheel_radius * caster_wheel_radius)}" iyz="0.0"
-            izz="${caster_wheel_mass * 0.4 * (caster_wheel_radius * caster_wheel_radius)}"/>
-        </inertial>
-      </link>
-      <joint name="${prefix}caster_rear_wheel_joint" type="continuous">
-        <parent link="${prefix}chassis_link"/>
-        <child link="${prefix}caster_rear_wheel"/>
-        <origin xyz="${-base_width/2 + caster_wheel_radius} 0 ${wheel_z_offset}" rpy="0 0 0"/>
-      </joint>
-      <link name="${prefix}caster_rear_wheel">
-        <collision>
-          <origin xyz="0 0 0" rpy="0 0 0"/>
-          <geometry>
-            <sphere radius="${caster_wheel_radius}"/>
-          </geometry>
-        </collision>
-        <visual>
-          <origin xyz="0 0 0" rpy="0 0 0"/>
-          <geometry>
-            <sphere radius="${caster_wheel_radius}"/>
-          </geometry>
-          <material name="white"/>
-        </visual>
-        <inertial>
-          <origin xyz="0 0 0" rpy="0 0 0"/>
-          <mass value="${caster_wheel_mass}"/>
-          <inertia
-            ixx="${caster_wheel_mass * 0.4 * (caster_wheel_radius * caster_wheel_radius)}" ixy="0.0" ixz="0.0"
-            iyy="${caster_wheel_mass * 0.4 * (caster_wheel_radius * caster_wheel_radius)}" iyz="0.0"
-            izz="${caster_wheel_mass * 0.4 * (caster_wheel_radius * caster_wheel_radius)}"/>
+      <joint name="${prefix}caster_left_wheel_joint" type="continuous">
+        <parent link="${prefix}chassis_link"/>
+        <child link="${prefix}caster_left_wheel"/>
+        <origin xyz="${-base_length/2} ${base_width/2} ${wheel_z_offset}" rpy="0 0 ${rear_left_wheel_yaw}"/>
+        <axis xyz="0 1 0"/>
+        <dynamics damping="0.05"/>
+        <limit effort="100" velocity="20.0"/>
+      </joint>
+      <link name="${prefix}caster_left_wheel">
+        <collision>
+          <origin xyz="0 0 0" rpy="${PI/2} 0 ${PI}"/>
+          <geometry>
+            <cylinder length="${wheel_len}" radius="${wheel_radius}"/>
+          </geometry>
+        </collision>
+        <visual>
+          <origin xyz="0 0 0" rpy="${PI/2} 0 ${PI}"/>
+          <geometry>
+            <!-- <cylinder length="${wheel_len}" radius="${wheel_radius}"/> -->
+            <mesh filename="package://studica_vmxpi_ros2/description/meshes/wheels/omni_wheel_v2.dae" scale="1.0 1.0 1.0"/>
+          </geometry>
+          <!-- <material name="black"/> -->
+        </visual>
+        <inertial>
+          <origin xyz="0 0 0" rpy="${PI/2} 0 ${PI}"/>
+          <mass value="${wheel_mass}"/>
+          <inertia
+            ixx="${wheel_mass / 12.0 * (3*wheel_radius*wheel_radius + wheel_len*wheel_len)}" ixy="0.0" ixz="0.0"
+            iyy="${wheel_mass / 12.0 * (3*wheel_radius*wheel_radius + wheel_len*wheel_len)}" iyz="0.0"
+            izz="${wheel_mass / 2.0 * wheel_radius*wheel_radius}"/>
+        </inertial>
+      </link>
+      <joint name="${prefix}caster_right_wheel_joint" type="continuous">
+        <parent link="${prefix}chassis_link"/>
+        <child link="${prefix}caster_right_wheel"/>
+        <origin xyz="${-base_length/2} -${base_width/2} ${wheel_z_offset}" rpy="0 0 ${rear_right_wheel_yaw}"/>
+        <axis xyz="0 1 0"/>
+        <dynamics damping="0.05"/>
+        <limit effort="100" velocity="20.0"/>
+      </joint>
+      <link name="${prefix}caster_right_wheel">
+         <collision>
+          <origin xyz="0 0 0" rpy="${PI/2} 0 0"/>
+          <geometry>
+            <cylinder length="${wheel_len}" radius="${wheel_radius}"/>
+          </geometry>
+        </collision>
+        <visual>
+          <origin xyz="0 0 0" rpy="${PI/2} 0 0"/>
+          <geometry>
+            <!-- <cylinder length="${wheel_len}" radius="${wheel_radius}"/> -->
+            <mesh filename="package://studica_vmxpi_ros2/description/meshes/wheels/omni_wheel_v2.dae" scale="1.0 1.0 1.0"/>
+          </geometry>
+          <!-- <material name="black"/> -->
+        </visual>
+        <inertial>
+          <origin xyz="0 0 0" rpy="${PI/2} 0 0"/>
+          <mass value="${wheel_mass}"/>
+          <inertia
+            ixx="${wheel_mass / 12.0 * (3*wheel_radius*wheel_radius + wheel_len*wheel_len)}" ixy="0.0" ixz="0.0"
+            iyy="${wheel_mass / 12.0 * (3*wheel_radius*wheel_radius + wheel_len*wheel_len)}" iyz="0.0"
+            izz="${wheel_mass / 2.0 * wheel_radius*wheel_radius}"/>
         </inertial>
       </link>
@@ -286,5 +294,4 @@
         <parent link="${prefix}chassis_link"/>
         <child link="${prefix}rear_right_wheel"/>
-        <!-- <origin xyz="${-base_length/2 + wheel_radius} -${base_width/2} ${wheel_z_offset}" rpy="0 0 ${rear_right_wheel_yaw}"/> -->
         <origin xyz="${-base_length/2} -${base_width/2} ${wheel_z_offset}" rpy="0 0 ${rear_right_wheel_yaw}"/>
         <axis xyz="0 1 0"/>

File: description/ros2_control/robot.ros2_control.xacro (robot description, xacro)
@@ -98,9 +98,9 @@
       <xacro:if value="${use_gz_sim and wheel_layout_resolved == 'diff'}">
         <!-- Gazebo Sim: publish passive caster joints so robot_state_publisher can build full TF tree. -->
-        <joint name="${prefix}caster_frontal_wheel_joint">
+        <joint name="${prefix}caster_left_wheel_joint">
           <state_interface name="position"/>
           <state_interface name="velocity"/>
         </joint>
-        <joint name="${prefix}caster_rear_wheel_joint">
+        <joint name="${prefix}caster_right_wheel_joint">
           <state_interface name="position"/>
           <state_interface name="velocity"/>
