Commit message: Improve gz_sim camera integration and add low-load performance controls

File: description/gz/robot.gz.xacro (robot description, xacro)
@@ -1,8 +1,10 @@
 <?xml version="1.0"?>
 <robot xmlns:xacro="http://ros.org/wiki/xacro">
-  <xacro:macro name="robot_gz" params="prefix gz_version controllers_file wheel_layout:=diff">
+  <xacro:macro name="robot_gz" params="prefix gz_version controllers_file wheel_layout:=diff sim_enable_camera:=true sim_camera_width:=640 sim_camera_height:=480 sim_camera_update_rate:=30.0 sim_lidar_samples:=200 sim_lidar_update_rate:=20.0 sim_lidar_visualize:=true sim_imu_update_rate:=100.0">
     <xacro:property name="wheel_layout_resolved" value="${wheel_layout if wheel_layout in ['diff', 'diff_4wd', 'mecanum', 'omni'] else 'diff'}"/>
     <xacro:property name="holonomic_mu1" value="${1.0 if wheel_layout_resolved == 'mecanum' else 4.0}"/>
     <xacro:property name="holonomic_mu2" value="${1.0 if wheel_layout_resolved == 'mecanum' else 4.0}"/>
+    <xacro:property name="sim_camera_enabled" value="${str(sim_enable_camera).lower() in ['true', '1', 'yes', 'on']}"/>
+    <xacro:property name="sim_lidar_visualize_enabled" value="${str(sim_lidar_visualize).lower() in ['true', '1', 'yes', 'on']}"/>
     <!-- ros2_control plugin for Gazebo Sim -->
     <xacro:if value="${int(gz_version) &lt; 7}">
@@ -118,10 +120,10 @@
         <topic>/scan</topic>
         <always_on>true</always_on>
-        <visualize>true</visualize>
-        <update_rate>20.0</update_rate>
+        <visualize>${sim_lidar_visualize_enabled}</visualize>
+        <update_rate>${sim_lidar_update_rate}</update_rate>
         <ray>
           <scan>
             <horizontal>
-              <samples>200</samples>
+              <samples>${sim_lidar_samples}</samples>
               <resolution>1</resolution>
               <min_angle>-3.14</min_angle>
@@ -143,8 +145,55 @@
         <topic>/imu</topic>
         <always_on>true</always_on>
-        <update_rate>100.0</update_rate>
+        <update_rate>${sim_imu_update_rate}</update_rate>
         <visualize>false</visualize>
       </sensor>
     </gazebo>
+    <!-- RGB + depth camera topics are bridged by ros_gz_bridge in gz_sim mode. -->
+    <xacro:if value="${sim_camera_enabled}">
+      <gazebo reference="${prefix}camera_link">
+        <sensor name="camera_color_sensor" type="camera">
+          <pose>0 0 0 0 0 0</pose>
+          <topic>/camera/color/image_raw</topic>
+          <always_on>true</always_on>
+          <visualize>false</visualize>
+          <update_rate>${sim_camera_update_rate}</update_rate>
+          <camera>
+            <camera_info_topic>/camera/color/camera_info</camera_info_topic>
+            <optical_frame_id>${prefix}camera_optical_frame</optical_frame_id>
+            <horizontal_fov>1.3962634</horizontal_fov>
+            <image>
+              <width>${sim_camera_width}</width>
+              <height>${sim_camera_height}</height>
+              <format>R8G8B8</format>
+            </image>
+            <clip>
+              <near>0.05</near>
+              <far>20.0</far>
+            </clip>
+          </camera>
+        </sensor>
+        <sensor name="camera_depth_sensor" type="depth_camera">
+          <pose>0 0 0 0 0 0</pose>
+          <topic>/camera/depth/image_raw</topic>
+          <always_on>true</always_on>
+          <visualize>false</visualize>
+          <update_rate>${sim_camera_update_rate}</update_rate>
+          <camera>
+            <camera_info_topic>/camera/depth/camera_info</camera_info_topic>
+            <optical_frame_id>${prefix}camera_optical_frame</optical_frame_id>
+            <horizontal_fov>1.3962634</horizontal_fov>
+            <image>
+              <width>${sim_camera_width}</width>
+              <height>${sim_camera_height}</height>
+              <format>R_FLOAT32</format>
+            </image>
+            <clip>
+              <near>0.05</near>
+              <far>20.0</far>
+            </clip>
+          </camera>
+        </sensor>
+      </gazebo>
+    </xacro:if>
   </xacro:macro>
 </robot>

File: description/robot/urdf/robot_description.urdf.xacro (robot description, xacro)
@@ -1,5 +1,5 @@
 <?xml version="1.0"?>
 <robot xmlns:xacro="http://www.ros.org/wiki/xacro">
-  <xacro:macro name="robot_description" params="prefix base_mass:=10.0 base_width:=0.4 base_length:=0.4 base_height:=0.1 wheel_mass:=0.3 wheel_len:=0.04 wheel_radius:=0.05 wheel_z_offset:=-0.027 caster_wheel_mass:=0.1 caster_wheel_radius:=0.05 laser1_model_x:=0.192 laser_model_z:=0.0 laser_frame_z:=0.03 wheel_layout:=diff">
+  <xacro:macro name="robot_description" params="prefix base_mass:=10.0 base_width:=0.4 base_length:=0.4 base_height:=0.1 wheel_mass:=0.3 wheel_len:=0.04 wheel_radius:=0.05 wheel_z_offset:=-0.027 caster_wheel_mass:=0.1 caster_wheel_radius:=0.05 laser_pos_x:=0.192 laser_pos_z:=0.0 laser_frame_z:=0.03 cam_pos_x:=${base_length/2.0} cam_pos_y:=0.0 cam_pos_z:=${base_height/2.0} cam_roll:=0.0 cam_pitch:=0.0 cam_yaw:=0.0 wheel_layout:=diff">
     <!-- Constants for robot dimensions -->
     <xacro:property name="PI" value="3.1415926535897931"/>
@@ -344,5 +344,5 @@
     </link>
     <joint name="${prefix}laser_scan_model_link_joint" type="fixed">
-      <origin rpy="0 0 0" xyz="${laser1_model_x} 0 ${laser_model_z}"/>
+      <origin rpy="0 0 0" xyz="${laser_pos_x} 0 ${laser_pos_z}"/>
       <parent link="${prefix}chassis_link"/>
       <child link="${prefix}laser_model_link"/>
@@ -365,4 +365,25 @@
       <child link="${prefix}imu_link"/>
     </joint>
+    <!-- Camera mounting frame used by Gazebo Sim camera sensors. -->
+    <link name="${prefix}camera_link">
+      <visual>
+        <origin xyz="0 0 0" rpy="0 0 0"/>
+        <geometry>
+          <mesh filename="package://studica_vmxpi_ros2/description/meshes/sensors/3d_depth_camera.dae" scale="1.0 1.0 1.0"/>
+        </geometry>
+      </visual>
+    </link>
+    <joint name="${prefix}camera_link_joint" type="fixed">
+      <origin rpy="${cam_roll} ${cam_pitch} ${cam_yaw}" xyz="${cam_pos_x} ${cam_pos_y} ${cam_pos_z}"/>
+      <parent link="${prefix}chassis_link"/>
+      <child link="${prefix}camera_link"/>
+    </joint>
+    <!-- ROS optical frame convention (REP-103): z forward, x right, y down. -->
+    <link name="${prefix}camera_optical_frame"/>
+    <joint name="${prefix}camera_optical_frame_joint" type="fixed">
+      <origin xyz="0 0 0" rpy="${-PI/2} 0 ${-PI/2}"/>
+      <parent link="${prefix}camera_link"/>
+      <child link="${prefix}camera_optical_frame"/>
+    </joint>
   </xacro:macro>
 </robot>

File: description/urdf/robot.urdf.xacro (robot description, xacro)
@@ -7,4 +7,12 @@
   <xacro:arg name="use_gz_sim" default="false" />
   <xacro:arg name="gz_version" default="8" />
+  <xacro:arg name="sim_enable_camera" default="true" />
+  <xacro:arg name="sim_camera_width" default="640" />
+  <xacro:arg name="sim_camera_height" default="480" />
+  <xacro:arg name="sim_camera_update_rate" default="30.0" />
+  <xacro:arg name="sim_lidar_samples" default="200" />
+  <xacro:arg name="sim_lidar_update_rate" default="20.0" />
+  <xacro:arg name="sim_lidar_visualize" default="true" />
+  <xacro:arg name="sim_imu_update_rate" default="100.0" />
   <xacro:arg name="profile_file" default="$(find studica_vmxpi_ros2)/config/profiles/training_4wd/robot_profile.yaml" />
   <xacro:arg name="controllers_file" default="$(find studica_vmxpi_ros2)/config/profiles/training_4wd/robot_controllers.yaml" />
@@ -18,4 +26,10 @@
   <xacro:property name="drive_cfg" value="${profile['drive'] if 'drive' in profile else dict()}"/>
   <xacro:property name="wheel_layout" value="${str(drive_cfg.get('wheel_layout', 'diff')).lower()}"/>
+  <xacro:property name="cam_pos_x" value="${geometry_cfg.get('cam_pos_x', geometry_cfg['base_length'] / 4.0)}"/>
+  <xacro:property name="cam_pos_y" value="${geometry_cfg.get('cam_pos_y', 0.0)}"/>
+  <xacro:property name="cam_pos_z" value="${geometry_cfg.get('cam_pos_z', geometry_cfg['base_height'] / 2.0)}"/>
+  <xacro:property name="cam_roll" value="${geometry_cfg.get('cam_roll', 0.0)}"/>
+  <xacro:property name="cam_pitch" value="${geometry_cfg.get('cam_pitch', 0.0)}"/>
+  <xacro:property name="cam_yaw" value="${geometry_cfg.get('cam_yaw', 0.0)}"/>
   <xacro:robot_description
     prefix="$(arg prefix)"
@@ -29,6 +43,12 @@
     caster_wheel_mass="${geometry_cfg['caster_wheel_mass']}"
     caster_wheel_radius="${geometry_cfg['caster_wheel_radius']}"
-    laser_model_z="${geometry_cfg['laser_model_z']}"
+    laser_pos_z="${geometry_cfg['laser_pos_z']}"
     laser_frame_z="${geometry_cfg['laser_frame_z']}"
+    cam_pos_x="${cam_pos_x}"
+    cam_pos_y="${cam_pos_y}"
+    cam_pos_z="${cam_pos_z}"
+    cam_roll="${cam_roll}"
+    cam_pitch="${cam_pitch}"
+    cam_yaw="${cam_yaw}"
     wheel_layout="${wheel_layout}"/>
   <xacro:robot_ros2_control
@@ -55,4 +75,12 @@
       gz_version="$(arg gz_version)"
       controllers_file="$(arg controllers_file)"
+      sim_enable_camera="$(arg sim_enable_camera)"
+      sim_camera_width="$(arg sim_camera_width)"
+      sim_camera_height="$(arg sim_camera_height)"
+      sim_camera_update_rate="$(arg sim_camera_update_rate)"
+      sim_lidar_samples="$(arg sim_lidar_samples)"
+      sim_lidar_update_rate="$(arg sim_lidar_update_rate)"
+      sim_lidar_visualize="$(arg sim_lidar_visualize)"
+      sim_imu_update_rate="$(arg sim_imu_update_rate)"
       wheel_layout="${wheel_layout}"/>
   </xacro:if>
