Commit message: Add real robot mapping and navigation workflows

File: description/gz/robot.gz.xacro (robot description, xacro)
@@ -140,5 +140,5 @@
     </gazebo>
     <!-- IMU publishes on Gazebo topic /imu; ros_gz_bridge forwards to ROS /imu -->
-    <gazebo reference="${prefix}chassis_link">
+    <gazebo reference="${prefix}imu_link">
       <sensor name="imu_sensor" type="imu">
         <pose>0 0 0 0 0 0</pose>

File: description/robot/urdf/robot_description.urdf.xacro (robot description, xacro)
@@ -1,9 +1,10 @@
 <?xml version="1.0"?>
 <robot xmlns:xacro="http://www.ros.org/wiki/xacro">
-  <xacro:macro name="robot_description" params="prefix wheel_radius base_mass:=10.0 base_width:=0.4 base_length:=0.4 base_height:=0.1 wheel_mass:=0.3 wheel_len:=0.04 wheel_z_offset:=-0.027 caster_wheel_mass:=0.1 caster_wheel_radius:=0.05 laser_pos_x:=0.192 laser_pos_z:=0.0 laser_frame_z:=0.03 cam_pos_x:=${base_length/2.0} cam_pos_y:=0.0 cam_pos_z:=${base_height/2.0} cam_roll:=0.0 cam_pitch:=0.0 cam_yaw:=0.0 wheel_layout:=diff">
+  <xacro:macro name="robot_description" params="prefix wheel_radius base_mass:=10.0 base_width:=0.4 base_length:=0.4 base_height:=0.1 chassis_center_z:=0.077 wheelbase:=${base_length} wheel_track:=${base_width} use_chassis_mesh:=true wheel_mass:=0.3 wheel_len:=0.04 caster_wheel_mass:=0.1 caster_wheel_radius:=0.05 laser_pos_x:=0.192 laser_pos_y:=0.0 laser_pos_z:=0.0 laser_roll:=0.0 laser_pitch:=0.0 laser_yaw:=0.0 laser_frame_z:=0.03 cam_pos_x:=${base_length/2.0} cam_pos_y:=0.0 cam_pos_z:=${base_height/2.0} cam_roll:=0.0 cam_pitch:=0.0 cam_yaw:=0.0 imu_pos_x:=0.0 imu_pos_y:=0.0 imu_pos_z:=0.0 imu_roll:=0.0 imu_pitch:=0.0 imu_yaw:=0.0 wheel_layout:=diff">
     <!-- Constants for robot dimensions -->
     <xacro:property name="PI" value="3.1415926535897931"/>
-    <!-- <xacro:property name="z_offset" value="${wheel_z_offset}"/> -->
     <xacro:property name="wheel_layout_resolved" value="${wheel_layout if wheel_layout in ['diff', 'diff_4wd', 'mecanum', 'omni'] else 'diff'}"/>
+    <xacro:property name="use_chassis_mesh_resolved" value="${str(use_chassis_mesh).lower() in ['true', '1', 'yes', 'on']}"/>
+    <xacro:property name="wheel_center_z" value="${float(wheel_radius) - float(chassis_center_z)}"/>
     <xacro:property name="front_left_wheel_yaw" value="${-PI/4 if wheel_layout_resolved == 'omni' else 0.0}"/>
     <xacro:property name="front_right_wheel_yaw" value="${PI/4 if wheel_layout_resolved == 'omni' else 0.0}"/>
@@ -11,5 +12,5 @@
     <xacro:property name="rear_right_wheel_yaw" value="${-PI/4 if wheel_layout_resolved == 'omni' else 0.0}"/>
     <!-- Keep base_link/base_footprint on the ground plane. -->
-    <xacro:property name="base_to_chassis_z" value="${float(wheel_radius) - float(wheel_z_offset)}"/>
+    <xacro:property name="base_to_chassis_z" value="${float(chassis_center_z)}"/>
     <xacro:if value="${wheel_layout_resolved == 'diff'}">
       <xacro:property name="robot_frame_mesh_file" value="package://studica_vmxpi_ros2/description/meshes/frames/robot_frame_4wd.dae"/>
@@ -38,6 +39,6 @@
         <origin xyz="0 0 0" rpy="0 0 0"/>
         <geometry>
-          <!-- Keep collision primitive simple/stable for physics engines (DART). -->
-          <box size="${base_length - wheel_len} ${base_width - wheel_len} ${base_height}"/>
+          <!-- Measured body envelope; keep collision primitive stable for DART. -->
+          <box size="${base_length} ${base_width} ${base_height}"/>
         </geometry>
       </collision>
@@ -45,8 +46,14 @@
         <origin xyz="0 0 0" rpy="0 0 0"/>
         <geometry>
-          <!-- <box size="${base_length} ${base_width} ${base_height}"/> -->
-          <mesh filename="${robot_frame_mesh_file}" scale="1.0 1.0 1.0"/>
+          <xacro:if value="${use_chassis_mesh_resolved}">
+            <mesh filename="${robot_frame_mesh_file}" scale="1.0 1.0 1.0"/>
+          </xacro:if>
+          <xacro:unless value="${use_chassis_mesh_resolved}">
+            <box size="${base_length} ${base_width} ${base_height}"/>
+          </xacro:unless>
         </geometry>
-        <!-- <material name="orange"/> -->
+        <xacro:unless value="${use_chassis_mesh_resolved}">
+          <material name="orange"/>
+        </xacro:unless>
       </visual>
       <inertial>
@@ -54,6 +61,6 @@
         <mass value="${base_mass}"/>
         <inertia
-          ixx="${base_mass / 12.0 * (base_length*base_length + base_height*base_height)}" ixy="0.0" ixz="0.0"
-          iyy="${base_mass / 12.0 * (base_height*base_height + base_width*base_width)}" iyz="0.0"
+          ixx="${base_mass / 12.0 * (base_width*base_width + base_height*base_height)}" ixy="0.0" ixz="0.0"
+          iyy="${base_mass / 12.0 * (base_length*base_length + base_height*base_height)}" iyz="0.0"
           izz="${base_mass / 12.0 * (base_width*base_width + base_length*base_length)}"/>
       </inertial>
@@ -68,5 +75,5 @@
         <parent link="${prefix}chassis_link"/>
         <child link="${prefix}left_wheel"/>
-        <origin xyz="${base_length/2} ${base_width/2} ${wheel_z_offset}" rpy="0 0 0"/>
+        <origin xyz="${wheelbase/2} ${wheel_track/2} ${wheel_center_z}" rpy="0 0 0"/>
         <axis xyz="0 1 0"/>
         <dynamics damping="0.05"/>
@@ -100,5 +107,5 @@
         <parent link="${prefix}chassis_link"/>
         <child link="${prefix}right_wheel"/>
-        <origin xyz="${base_length/2} -${base_width/2} ${wheel_z_offset}" rpy="0 0 0"/>
+        <origin xyz="${wheelbase/2} -${wheel_track/2} ${wheel_center_z}" rpy="0 0 0"/>
         <axis xyz="0 1 0"/>
         <dynamics damping="0.05"/>
@@ -132,5 +139,5 @@
         <parent link="${prefix}chassis_link"/>
         <child link="${prefix}caster_left_wheel"/>
-        <origin xyz="${-base_length/2} ${base_width/2} ${wheel_z_offset}" rpy="0 0 ${rear_left_wheel_yaw}"/>
+        <origin xyz="${-wheelbase/2} ${wheel_track/2} ${wheel_center_z}" rpy="0 0 ${rear_left_wheel_yaw}"/>
         <axis xyz="0 1 0"/>
         <dynamics damping="0.05"/>
@@ -164,5 +171,5 @@
         <parent link="${prefix}chassis_link"/>
         <child link="${prefix}caster_right_wheel"/>
-        <origin xyz="${-base_length/2} -${base_width/2} ${wheel_z_offset}" rpy="0 0 ${rear_right_wheel_yaw}"/>
+        <origin xyz="${-wheelbase/2} -${wheel_track/2} ${wheel_center_z}" rpy="0 0 ${rear_right_wheel_yaw}"/>
         <axis xyz="0 1 0"/>
         <dynamics damping="0.05"/>
@@ -198,5 +205,5 @@
         <parent link="${prefix}chassis_link"/>
         <child link="${prefix}front_left_wheel"/>
-        <origin xyz="${base_length/2} ${base_width/2} ${wheel_z_offset}" rpy="0 0 ${front_left_wheel_yaw}"/>
+        <origin xyz="${wheelbase/2} ${wheel_track/2} ${wheel_center_z}" rpy="0 0 ${front_left_wheel_yaw}"/>
         <axis xyz="0 1 0"/>
         <dynamics damping="0.05"/>
@@ -230,5 +237,5 @@
         <parent link="${prefix}chassis_link"/>
         <child link="${prefix}front_right_wheel"/>
-        <origin xyz="${base_length/2} -${base_width/2} ${wheel_z_offset}" rpy="0 0 ${front_right_wheel_yaw}"/>
+        <origin xyz="${wheelbase/2} -${wheel_track/2} ${wheel_center_z}" rpy="0 0 ${front_right_wheel_yaw}"/>
         <axis xyz="0 1 0"/>
         <dynamics damping="0.05"/>
@@ -262,5 +269,5 @@
         <parent link="${prefix}chassis_link"/>
         <child link="${prefix}rear_left_wheel"/>
-        <origin xyz="${-base_length/2} ${base_width/2} ${wheel_z_offset}" rpy="0 0 ${rear_left_wheel_yaw}"/>
+        <origin xyz="${-wheelbase/2} ${wheel_track/2} ${wheel_center_z}" rpy="0 0 ${rear_left_wheel_yaw}"/>
         <axis xyz="0 1 0"/>
         <dynamics damping="0.05"/>
@@ -294,5 +301,5 @@
         <parent link="${prefix}chassis_link"/>
         <child link="${prefix}rear_right_wheel"/>
-        <origin xyz="${-base_length/2} -${base_width/2} ${wheel_z_offset}" rpy="0 0 ${rear_right_wheel_yaw}"/>
+        <origin xyz="${-wheelbase/2} -${wheel_track/2} ${wheel_center_z}" rpy="0 0 ${rear_right_wheel_yaw}"/>
         <axis xyz="0 1 0"/>
         <dynamics damping="0.05"/>
@@ -344,5 +351,7 @@
     </link>
     <joint name="${prefix}laser_scan_model_link_joint" type="fixed">
-      <origin rpy="0 0 0" xyz="${laser_pos_x} 0 ${laser_pos_z}"/>
+      <origin
+        rpy="${laser_roll} ${laser_pitch} ${laser_yaw}"
+        xyz="${laser_pos_x} ${laser_pos_y} ${laser_pos_z}"/>
       <parent link="${prefix}chassis_link"/>
       <child link="${prefix}laser_model_link"/>
@@ -361,5 +370,7 @@
     </link>
     <joint name="${prefix}imu_link_joint" type="fixed">
-      <origin rpy="0 0 0" xyz="0 0 0"/>
+      <origin
+        rpy="${imu_roll} ${imu_pitch} ${imu_yaw}"
+        xyz="${imu_pos_x} ${imu_pos_y} ${imu_pos_z}"/>
       <parent link="${prefix}chassis_link"/>
       <child link="${prefix}imu_link"/>

File: description/urdf/robot.urdf.xacro (robot description, xacro)
@@ -25,4 +25,17 @@
   <xacro:property name="drive_cfg" value="${profile['drive'] if 'drive' in profile else dict()}"/>
   <xacro:property name="wheel_layout" value="${str(drive_cfg.get('wheel_layout', 'diff')).lower()}"/>
+  <xacro:property name="wheel_radius" value="${float(drive_cfg['wheel_radius_m'])}"/>
+  <xacro:property name="legacy_wheel_z_offset" value="${float(geometry_cfg.get('wheel_z_offset', -0.027))}"/>
+  <xacro:property name="chassis_center_z" value="${float(geometry_cfg['ground_clearance']) + float(geometry_cfg['base_height']) / 2.0 if 'ground_clearance' in geometry_cfg else wheel_radius - legacy_wheel_z_offset}"/>
+  <xacro:property name="wheelbase" value="${geometry_cfg.get('wheelbase', geometry_cfg['base_length'])}"/>
+  <xacro:property name="wheel_track" value="${geometry_cfg.get('wheel_track', geometry_cfg['base_width'])}"/>
+  <xacro:property name="use_chassis_mesh" value="${geometry_cfg.get('use_chassis_mesh', True)}"/>
+  <xacro:property name="laser_pos_x" value="${geometry_cfg.get('laser_pos_x', 0.192)}"/>
+  <xacro:property name="laser_pos_y" value="${geometry_cfg.get('laser_pos_y', 0.0)}"/>
+  <xacro:property name="laser_pos_z" value="${geometry_cfg.get('laser_pos_z', 0.0)}"/>
+  <xacro:property name="laser_roll" value="${geometry_cfg.get('laser_roll', 0.0)}"/>
+  <xacro:property name="laser_pitch" value="${geometry_cfg.get('laser_pitch', 0.0)}"/>
+  <xacro:property name="laser_yaw" value="${geometry_cfg.get('laser_yaw', 0.0)}"/>
+  <xacro:property name="laser_frame_z" value="${geometry_cfg.get('laser_frame_z', 0.03)}"/>
   <xacro:property name="cam_pos_x" value="${geometry_cfg.get('cam_pos_x', geometry_cfg['base_length'] / 4.0)}"/>
   <xacro:property name="cam_pos_y" value="${geometry_cfg.get('cam_pos_y', 0.0)}"/>
@@ -31,4 +44,10 @@
   <xacro:property name="cam_pitch" value="${geometry_cfg.get('cam_pitch', 0.0)}"/>
   <xacro:property name="cam_yaw" value="${geometry_cfg.get('cam_yaw', 0.0)}"/>
+  <xacro:property name="imu_pos_x" value="${geometry_cfg.get('imu_pos_x', 0.0)}"/>
+  <xacro:property name="imu_pos_y" value="${geometry_cfg.get('imu_pos_y', 0.0)}"/>
+  <xacro:property name="imu_pos_z" value="${geometry_cfg.get('imu_pos_z', 0.0)}"/>
+  <xacro:property name="imu_roll" value="${geometry_cfg.get('imu_roll', 0.0)}"/>
+  <xacro:property name="imu_pitch" value="${geometry_cfg.get('imu_pitch', 0.0)}"/>
+  <xacro:property name="imu_yaw" value="${geometry_cfg.get('imu_yaw', 0.0)}"/>
   <xacro:robot_description
     prefix="$(arg prefix)"
@@ -37,11 +56,20 @@
     base_length="${geometry_cfg['base_length']}"
     base_height="${geometry_cfg['base_height']}"
+    chassis_center_z="${chassis_center_z}"
+    wheelbase="${wheelbase}"
+    wheel_track="${wheel_track}"
+    use_chassis_mesh="${use_chassis_mesh}"
     wheel_mass="${geometry_cfg['wheel_mass']}"
     wheel_len="${geometry_cfg['wheel_len']}"
-    wheel_radius="${drive_cfg['wheel_radius_m']}"
+    wheel_radius="${wheel_radius}"
     caster_wheel_mass="${geometry_cfg['caster_wheel_mass']}"
     caster_wheel_radius="${geometry_cfg['caster_wheel_radius']}"
-    laser_pos_z="${geometry_cfg['laser_pos_z']}"
-    laser_frame_z="${geometry_cfg['laser_frame_z']}"
+    laser_pos_x="${laser_pos_x}"
+    laser_pos_y="${laser_pos_y}"
+    laser_pos_z="${laser_pos_z}"
+    laser_roll="${laser_roll}"
+    laser_pitch="${laser_pitch}"
+    laser_yaw="${laser_yaw}"
+    laser_frame_z="${laser_frame_z}"
     cam_pos_x="${cam_pos_x}"
     cam_pos_y="${cam_pos_y}"
@@ -50,4 +78,10 @@
     cam_pitch="${cam_pitch}"
     cam_yaw="${cam_yaw}"
+    imu_pos_x="${imu_pos_x}"
+    imu_pos_y="${imu_pos_y}"
+    imu_pos_z="${imu_pos_z}"
+    imu_roll="${imu_roll}"
+    imu_pitch="${imu_pitch}"
+    imu_yaw="${imu_yaw}"
     wheel_layout="${wheel_layout}"/>
   <xacro:robot_ros2_control
