Commit message: Remove Gazebo Classic support and stabilize Nav2 simulation bringup

File: description/ros2_control/robot.ros2_control.xacro (robot description, xacro)
@@ -1,14 +1,9 @@
 <?xml version="1.0"?>
 <robot xmlns:xacro="http://www.ros.org/wiki/xacro">
-  <xacro:macro name="robot_ros2_control" params="name prefix use_hardware use_gazebo_classic use_gz_sim profile_file wheel_layout:=diff">
+  <xacro:macro name="robot_ros2_control" params="name prefix use_hardware use_gz_sim profile_file wheel_layout:=diff">
     <xacro:property name="profile" value="${xacro.load_yaml(profile_file)}"/>
     <xacro:property name="hardware_cfg" value="${profile['hardware']}"/>
     <xacro:property name="wheel_layout_resolved" value="${wheel_layout if wheel_layout in ['diff', 'diff_4wd', 'mecanum', 'omni'] else 'diff'}"/>
     <ros2_control name="${name}" type="system">
-      <xacro:if value="${use_gazebo_classic}">
-        <hardware>
-          <plugin>gazebo_ros2_control/GazeboSystem</plugin>
-        </hardware>
-      </xacro:if>
       <xacro:if value="${use_gz_sim}">
         <hardware>
@@ -16,5 +11,5 @@
         </hardware>
       </xacro:if>
-      <xacro:unless value="${use_gazebo_classic or use_gz_sim}">
+      <xacro:unless value="${use_gz_sim}">
       <xacro:if value="${use_hardware}">
         <hardware>
@@ -82,5 +77,5 @@
         </joint>
       </xacro:unless>
-      <xacro:if value="${use_hardware and not use_gazebo_classic and not use_gz_sim}">
+      <xacro:if value="${use_hardware and not use_gz_sim}">
         <sensor name="imu_sensor">
           <state_interface name="orientation.x"/>

File: description/urdf/robot.urdf.xacro (robot description, xacro)
@@ -4,5 +4,4 @@
   <xacro:arg name="prefix" default="" />
   <xacro:arg name="use_hardware" default="false" />
-  <xacro:arg name="use_gazebo_classic" default="false" />
   <xacro:arg name="use_gz_sim" default="false" />
   <xacro:arg name="gz_version" default="8" />
@@ -56,16 +55,7 @@
     prefix="$(arg prefix)"
     use_hardware="$(arg use_hardware)"
-    use_gazebo_classic="$(arg use_gazebo_classic)"
     use_gz_sim="$(arg use_gz_sim)"
     profile_file="$(arg profile_file)"
     wheel_layout="${wheel_layout}"/>
-  <xacro:if value="$(arg use_gazebo_classic)">
-    <!-- Import Gazebo Classic definitions + plugin -->
-    <xacro:include filename="$(find studica_vmxpi_ros2)/description/gazebo/robot.gazebo.xacro" />
-    <xacro:robot_gazebo
-      prefix="$(arg prefix)"
-      controllers_file="$(arg controllers_file)"
-      wheel_layout="${wheel_layout}"/>
-  </xacro:if>
   <xacro:if value="$(arg use_gz_sim)">
     <!-- Import Gazebo Sim definitions + plugin -->
