Commit message: feat: add Titan velocity PID and Foxglove health dashboard

File: description/robot/urdf/robot_description.urdf.xacro (robot description, xacro)
@@ -1,5 +1,5 @@
 <?xml version="1.0"?>
 <robot xmlns:xacro="http://www.ros.org/wiki/xacro">
-  <xacro:macro name="robot_description" params="prefix base_mass:=10.0 base_width:=0.4 base_length:=0.4 base_height:=0.1 wheel_mass:=0.3 wheel_len:=0.04 wheel_radius:=0.05 wheel_z_offset:=-0.027 caster_wheel_mass:=0.1 caster_wheel_radius:=0.05 laser_pos_x:=0.192 laser_pos_z:=0.0 laser_frame_z:=0.03 cam_pos_x:=${base_length/2.0} cam_pos_y:=0.0 cam_pos_z:=${base_height/2.0} cam_roll:=0.0 cam_pitch:=0.0 cam_yaw:=0.0 wheel_layout:=diff">
+  <xacro:macro name="robot_description" params="prefix wheel_radius base_mass:=10.0 base_width:=0.4 base_length:=0.4 base_height:=0.1 wheel_mass:=0.3 wheel_len:=0.04 wheel_z_offset:=-0.027 caster_wheel_mass:=0.1 caster_wheel_radius:=0.05 laser_pos_x:=0.192 laser_pos_z:=0.0 laser_frame_z:=0.03 cam_pos_x:=${base_length/2.0} cam_pos_y:=0.0 cam_pos_z:=${base_height/2.0} cam_roll:=0.0 cam_pitch:=0.0 cam_yaw:=0.0 wheel_layout:=diff">
     <!-- Constants for robot dimensions -->
     <xacro:property name="PI" value="3.1415926535897931"/>

File: description/ros2_control/robot.ros2_control.xacro (robot description, xacro)
@@ -4,4 +4,6 @@
     <xacro:property name="profile" value="${xacro.load_yaml(profile_file)}"/>
     <xacro:property name="hardware_cfg" value="${profile['hardware']}"/>
+    <xacro:property name="drive_cfg" value="${profile['drive']}"/>
+    <xacro:property name="pid_cfg" value="${hardware_cfg.get('pid', dict())}"/>
     <xacro:property name="wheel_layout_resolved" value="${wheel_layout if wheel_layout in ['diff', 'diff_4wd', 'mecanum', 'omni'] else 'diff'}"/>
     <ros2_control name="${name}" type="system">
@@ -18,7 +20,16 @@
           <param name="motor_freq">${hardware_cfg['motor_freq']}</param>
           <param name="ticks_per_rotation">${hardware_cfg['ticks_per_rotation']}</param>
-          <param name="wheel_radius">${hardware_cfg['wheel_radius']}</param>
+          <param name="wheel_radius">${drive_cfg['wheel_radius_m']}</param>
           <param name="speed_scale">${hardware_cfg['speed_scale']}</param>
           <param name="max_wheel_angular_velocity_rad_s">${hardware_cfg['max_wheel_angular_velocity_rad_s']}</param>
+          <param name="control_mode">${hardware_cfg.get('control_mode', 'open_loop')}</param>
+          <param name="pid_type">${pid_cfg.get('type', 'mcv2')}</param>
+          <param name="pid_sensitivity">${pid_cfg.get('sensitivity', 5)}</param>
+          <param name="pid_require_supported">${pid_cfg.get('require_supported', True)}</param>
+          <param name="feedback_warn_timeout_ms">${hardware_cfg.get('feedback_warn_timeout_ms', 100)}</param>
+          <param name="feedback_error_timeout_ms">${hardware_cfg.get('feedback_error_timeout_ms', 250)}</param>
+          <param name="controller_temp_error_c">${hardware_cfg.get('controller_temp_error_c', 80.0)}</param>
+          <param name="controller_temp_error_timeout_ms">${hardware_cfg.get('controller_temp_error_timeout_ms', 3000)}</param>
+          <param name="wheel_radius_calibrated">${hardware_cfg.get('wheel_radius_calibrated', True)}</param>
           <param name="left_front_motor">${hardware_cfg['left_front_motor']}</param>
           <param name="left_rear_motor">${hardware_cfg['left_rear_motor']}</param>
@@ -48,4 +59,10 @@
           <state_interface name="position"/>
           <state_interface name="velocity"/>
+          <xacro:if value="${use_hardware and not use_gz_sim}">
+            <state_interface name="commanded_velocity"/>
+            <state_interface name="feedback_age"/>
+            <state_interface name="encoder_fresh"/>
+            <state_interface name="command_saturated"/>
+          </xacro:if>
         </joint>
         <joint name="${prefix}right_wheel_joint">
@@ -53,4 +70,10 @@
           <state_interface name="position"/>
           <state_interface name="velocity"/>
+          <xacro:if value="${use_hardware and not use_gz_sim}">
+            <state_interface name="commanded_velocity"/>
+            <state_interface name="feedback_age"/>
+            <state_interface name="encoder_fresh"/>
+            <state_interface name="command_saturated"/>
+          </xacro:if>
         </joint>
       </xacro:if>
@@ -60,4 +83,10 @@
           <state_interface name="position"/>
           <state_interface name="velocity"/>
+          <xacro:if value="${use_hardware and not use_gz_sim}">
+            <state_interface name="commanded_velocity"/>
+            <state_interface name="feedback_age"/>
+            <state_interface name="encoder_fresh"/>
+            <state_interface name="command_saturated"/>
+          </xacro:if>
         </joint>
         <joint name="${prefix}front_right_wheel_joint">
@@ -65,4 +94,10 @@
           <state_interface name="position"/>
           <state_interface name="velocity"/>
+          <xacro:if value="${use_hardware and not use_gz_sim}">
+            <state_interface name="commanded_velocity"/>
+            <state_interface name="feedback_age"/>
+            <state_interface name="encoder_fresh"/>
+            <state_interface name="command_saturated"/>
+          </xacro:if>
         </joint>
         <joint name="${prefix}rear_left_wheel_joint">
@@ -70,4 +105,10 @@
           <state_interface name="position"/>
           <state_interface name="velocity"/>
+          <xacro:if value="${use_hardware and not use_gz_sim}">
+            <state_interface name="commanded_velocity"/>
+            <state_interface name="feedback_age"/>
+            <state_interface name="encoder_fresh"/>
+            <state_interface name="command_saturated"/>
+          </xacro:if>
         </joint>
         <joint name="${prefix}rear_right_wheel_joint">
@@ -75,7 +116,23 @@
           <state_interface name="position"/>
           <state_interface name="velocity"/>
+          <xacro:if value="${use_hardware and not use_gz_sim}">
+            <state_interface name="commanded_velocity"/>
+            <state_interface name="feedback_age"/>
+            <state_interface name="encoder_fresh"/>
+            <state_interface name="command_saturated"/>
+          </xacro:if>
         </joint>
       </xacro:unless>
       <xacro:if value="${use_hardware and not use_gz_sim}">
+        <sensor name="titan_controller">
+          <state_interface name="controller_temperature"/>
+          <state_interface name="temperature_age"/>
+          <state_interface name="pid_supported"/>
+          <state_interface name="pid_type"/>
+          <state_interface name="fault_latched"/>
+          <state_interface name="firmware_major"/>
+          <state_interface name="firmware_minor"/>
+          <state_interface name="firmware_patch"/>
+        </sensor>
         <sensor name="imu_sensor">
           <state_interface name="orientation.x"/>

File: description/urdf/robot.urdf.xacro (robot description, xacro)
@@ -39,5 +39,5 @@
     wheel_mass="${geometry_cfg['wheel_mass']}"
     wheel_len="${geometry_cfg['wheel_len']}"
-    wheel_radius="${geometry_cfg['wheel_radius']}"
+    wheel_radius="${drive_cfg['wheel_radius_m']}"
     caster_wheel_mass="${geometry_cfg['caster_wheel_mass']}"
     caster_wheel_radius="${geometry_cfg['caster_wheel_radius']}"

Commit message: feat: add stack_4wd navigation and raw depth workflow

File: description/robot/urdf/robot_description.urdf.xacro (robot description, xacro)
@@ -1,5 +1,5 @@
 <?xml version="1.0"?>
 <robot xmlns:xacro="http://www.ros.org/wiki/xacro">
-  <xacro:macro name="robot_description" params="prefix wheel_radius base_mass:=10.0 base_width:=0.4 base_length:=0.4 base_height:=0.1 chassis_center_z:=0.077 wheelbase:=${base_length} wheel_track:=${base_width} use_chassis_mesh:=true wheel_mass:=0.3 wheel_len:=0.04 caster_wheel_mass:=0.1 caster_wheel_radius:=0.05 laser_pos_x:=0.192 laser_pos_y:=0.0 laser_pos_z:=0.0 laser_roll:=0.0 laser_pitch:=0.0 laser_yaw:=0.0 laser_frame_z:=0.03 cam_pos_x:=${base_length/2.0} cam_pos_y:=0.0 cam_pos_z:=${base_height/2.0} cam_roll:=0.0 cam_pitch:=0.0 cam_yaw:=0.0 imu_pos_x:=0.0 imu_pos_y:=0.0 imu_pos_z:=0.0 imu_roll:=0.0 imu_pitch:=0.0 imu_yaw:=0.0 wheel_layout:=diff">
+  <xacro:macro name="robot_description" params="prefix wheel_radius base_mass:=10.0 base_width:=0.4 base_length:=0.4 base_height:=0.1 chassis_center_z:=0.077 wheelbase:=${base_length} wheel_track:=${base_width} use_chassis_mesh:=true chassis_mesh_scale:=1.0 wheel_mass:=0.3 wheel_len:=0.04 caster_wheel_mass:=0.1 caster_wheel_radius:=0.05 laser_pos_x:=0.192 laser_pos_y:=0.0 laser_pos_z:=0.0 laser_roll:=0.0 laser_pitch:=0.0 laser_yaw:=0.0 laser_frame_z:=0.03 cam_pos_x:=${base_length/2.0} cam_pos_y:=0.0 cam_pos_z:=${base_height/2.0} cam_roll:=0.0 cam_pitch:=0.0 cam_yaw:=0.0 imu_pos_x:=0.0 imu_pos_y:=0.0 imu_pos_z:=0.0 imu_roll:=0.0 imu_pitch:=0.0 imu_yaw:=0.0 wheel_layout:=diff">
     <!-- Constants for robot dimensions -->
     <xacro:property name="PI" value="3.1415926535897931"/>
@@ -47,5 +47,5 @@
         <geometry>
           <xacro:if value="${use_chassis_mesh_resolved}">
-            <mesh filename="${robot_frame_mesh_file}" scale="1.0 1.0 1.0"/>
+            <mesh filename="${robot_frame_mesh_file}" scale="${chassis_mesh_scale} ${chassis_mesh_scale} ${chassis_mesh_scale}"/>
           </xacro:if>
           <xacro:unless value="${use_chassis_mesh_resolved}">

File: description/urdf/robot.urdf.xacro (robot description, xacro)
@@ -31,4 +31,5 @@
   <xacro:property name="wheel_track" value="${geometry_cfg.get('wheel_track', geometry_cfg['base_width'])}"/>
   <xacro:property name="use_chassis_mesh" value="${geometry_cfg.get('use_chassis_mesh', True)}"/>
+  <xacro:property name="chassis_mesh_scale" value="${float(geometry_cfg.get('chassis_mesh_scale', 1.0))}"/>
   <xacro:property name="laser_pos_x" value="${geometry_cfg.get('laser_pos_x', 0.192)}"/>
   <xacro:property name="laser_pos_y" value="${geometry_cfg.get('laser_pos_y', 0.0)}"/>
@@ -60,4 +61,5 @@
     wheel_track="${wheel_track}"
     use_chassis_mesh="${use_chassis_mesh}"
+    chassis_mesh_scale="${chassis_mesh_scale}"
     wheel_mass="${geometry_cfg['wheel_mass']}"
     wheel_len="${geometry_cfg['wheel_len']}"
